File: MPPT_charger_20A.kicad_pcb (KiCad board)
At the start: 2 copper layers, 114.5 x 60.5 mm, 152 parts, among them J1 SOLAR, J2 LOAD, J3 BAT, J4 UEXT, J5 CONN_01X03, P1 CONN_01X02, P3 USB Micro B, Q1 CSD18540Q5B, Q2 CSD18540Q5B, Q3 CSD18540Q5B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

Commit message: Update to KiCad 5 schematic library
Parts:
- removed LOGO? (x2): LOGO-S_PLACE_M, LibreSolar:Watterott_Logo
- removed REF***: WEEE-Logo_4.2x6mm_SilkScreen, Symbols:WEEE-Logo_4.2x6mm_SilkScreen
- C1, C2: footprint Capacitors_THT:CP_Radial_D16.0mm_P7.50mm -> Capacitor_THT:CP_Radial_D16.0mm_P7.50mm
- C5: footprint Capacitors_THT:CP_Radial_D10.0mm_P5.00mm -> Capacitor_THT:CP_Radial_D10.0mm_P5.00mm
- D2: footprint Diodes_SMD:D_PowerDI-123 -> Diode_SMD:D_PowerDI-123
- JP3: footprint Pin_Headers:Pin_Header_Angled_1x02_Pitch2.54mm -> Connector_PinHeader_2.54mm:PinHeader_1x02_P2.54mm_Horizontal
- L2: footprint Inductors_SMD:L_0805 -> Inductor_SMD:L_0805_2012Metric
- L4: footprint Inductors_SMD:L_0603 -> Inductor_SMD:L_0603_1608Metric
- LED1, LED2: footprint LEDs:LED_0603 -> LED_SMD:LED_0603_1608Metric
- LOGO2: footprint Symbols:OSHW-Logo_5.7x6mm_SilkScreen -> Symbol:OSHW-Logo_5.7x6mm_SilkScreen
- MK1, MK2, MK3: footprint Mounting_Holes:MountingHole_3.2mm_M3 -> MountingHole:MountingHole_3.2mm_M3
- P1: footprint Pin_Headers:Pin_Header_Straight_1x02_Pitch2.54mm -> Connector_PinHeader_2.54mm:PinHeader_1x02_P2.54mm_Vertical
- SWD1: footprint Pin_Headers:Pin_Header_Straight_1x06_Pitch2.54mm -> Connector_PinHeader_2.54mm:PinHeader_1x06_P2.54mm_Vertical
- U2: footprint Housings_QFP:LQFP-48_7x7mm_Pitch0.5mm -> Package_QFP:LQFP-48_7x7mm_P0.5mm
- U3: footprint TO_SOT_Packages_SMD:SOT-223-3Lead_TabPin2 -> Package_TO_SOT_SMD:SOT-223-3_TabPin2
- U6: footprint TO_SOT_Packages_SMD:SOT-23-5 -> LibreSolar:SOT-23-5
Other:
- board text removed: "watterott.com"
