File: power_supply.sch (KiCad schematic (older format))
At the start: 24 parts, among them U4 MCP16331-CH, U5 AP2210-3.3, U6 LM2665

Commit message: Updated R/C/L symbols to IEC 60617 style
Parts:
- D2: symbol D_Schottky_ALT -> D_Schottky; ALT (none) -> DFLS160-7
- D5: symbol D_ALT -> D
- D7: symbol D_Schottky_ALT -> D_Schottky
- L3: ALT (none) -> WE-TPC-4818 744042220
- U5: ALT (none) -> MIC5225
Connections:
- wire segments 73 -> 72
Other:
- note added: "Choose between PV or \nbattery as power supply\ninput (default: battery)"
- note added: "Max current \noutput: 150mA"
- note removed: "(or DFLS160-7)"
- note removed: "C_in: TDK C3225X7R2A225K230AB\nC_out: Murata GRM21BR60J226ME39L\nL_filter: Murata LQM21PN4R7NGRD"
- note removed: "Choose between PV or battery as\npower supply input (default: battery)"
- note removed: "Inductor:\nWE-TPC-4818 744042220\nor Bourns SRR4028-220Y"
- note removed: "Max current \noutput: 150mA\nAlternative: MIC5225"
- note removed: "Murata GRM21BR61E106KA73L\n10uF, 25V, X5R"
- note removed: "Power supply"
- moved on the sheet: C14, C15, C19, C20, C21, C22, C23, C24, C35, C37, C38, C41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

Commit message: Updated revision: 0.8
Parts:
- removed C22: 1u, Capacitors_SMD:C_0603, symbol C
- removed C37: 10u, Capacitors_SMD:C_0805, symbol C
- removed D5: 1N4148W-7-F, Diodes_SMD:D_SOD-123, symbol D
- removed D7: SS16FP, Diodes_SMD:D_PowerDI-123, symbol D_Schottky
- removed R33, R38: 0, Resistors_SMD:R_0603, symbol R
- removed U6: LM2665, TO_SOT_Packages_SMD:SOT-23-6, symbol LM2665
- added U3: AZ1117, TO_SOT_Packages_SMD:SOT-223-3Lead_TabPin2, symbol AZ1117
- C14: footprint Capacitors_SMD:C_0805 -> LibreSolar:C_0805_2012; Comment (none) -> 100V, X7S; MFR Murata -> (none); MPN GRJ21BC72A105KE11L -> (none); Manufacturer (none) -> Murata; PartNumber (none) -> GRJ21BC72A105KE11L
- C15: value 4.7u -> 2.2u; footprint Capacitors_SMD:C_1206 -> LibreSolar:C_1210_3225; Alternative (none) -> TY HMK325B7225KN-T; Comment (none) -> 100V, X7R; MFR TDK -> (none); MPN C3225X7R2A225K230AB -> (none); Manufacturer (none) -> Murata; PartNumber (none) -> GRM31CR72A225KA73L
- C19, C41: footprint Capacitors_SMD:C_0603 -> LibreSolar:C_0603_1608; MFR Murata -> (none); MPN GRM188R71H104KA93D -> (none); Manufacturer (none) -> Murata; PartNumber (none) -> GRM188R71H104KA93D
- C20, C21, C24: footprint Capacitors_SMD:C_0805 -> LibreSolar:C_0805_2012; MFR Murata -> (none); MPN GRM21BR61E106KA73L -> (none); Manufacturer (none) -> Murata; PartNumber (none) -> GRM21BR61E106KA73L
- C23: footprint Capacitors_SMD:C_0603 -> LibreSolar:C_0603_1608; MFR Murata -> (none); MPN GRM188R61E105KA12D -> (none); Manufacturer (none) -> Murata; PartNumber (none) -> GRM188R61E105KA12D; Remarks (none) -> 25V
- C35: footprint Capacitors_SMD:C_0603 -> LibreSolar:C_0603_1608; MFR Murata -> (none); MPN GRM1885C2A101JA01D -> (none); Manufacturer (none) -> Murata; PartNumber (none) -> GRM1885C2A101JA01D
- C38: footprint Capacitors_SMD:C_0603 -> LibreSolar:C_0603_1608; MFR Murata -> (none); MPN GRM188R60J225KE19D -> (none); Manufacturer (none) -> Murata; PartNumber (none) -> GRM188R60J225KE19D
- D2: MFR Diodes Inc. -> (none); MPN SS16FP -> (none); Manufacturer (none) -> Diodes Inc.; PartNumber (none) -> SS16FP
- L2: MFR Murata -> (none); MPN LQM21PN4R7NGRD -> (none); Manufacturer (none) -> Murata; PartNumber (none) -> LQM21PN4R7NGRD
- L3: value 22uH -> 47uH; footprint Inductors:SELF-WE-TPC_M -> LibreSolar:L_Wuerth_WE-TPC-58xx; ALT WE-TPC-4818 744042220 -> (none); Alternative (none) -> WE-TPC-5828 744053470; MFR Bourns -> (none); MPN SRR4028-220Y -> (none); Manufacturer (none) -> Bourns; PartNumber (none) -> SRR5028-470Y
- R28: value 52.3k -> 120k; footprint Resistors_SMD:R_0603 -> LibreSolar:R_0603_1608; MFR Yageo -> (none); MPN RC0603FR-0752K3L -> (none); Manufacturer (none) -> Yageo; PartNumber (none) -> RC0603FR-07120KL
- R29: footprint Resistors_SMD:R_0603 -> LibreSolar:R_0603_1608; MFR Yageo -> (none); MPN RC0603FR-07150KL -> (none); Manufacturer (none) -> Yageo; PartNumber (none) -> RC0603FR-07150KL
- U4: value MCP16331-CH -> LMR16006X; footprint TO_SOT_Packages_SMD:SOT-23-6 -> LibreSolar:SOT-23-6; symbol MCP16331-CH -> LMR16006; MFR Microchip -> (none); MPN MCP16331T-E/CH -> (none); Manufacturer (none) -> Texas Instruments; PartNumber (none) -> LMR16006X
- U5: footprint TO_SOT_Packages_SMD:SOT-23-5 -> LibreSolar:SOT-23-5; MFR Diodes Inc. -> (none); MPN AP2210K-3.3TRG1 -> (none); Manufacturer (none) -> Diodes Inc.; PartNumber (none) -> AP2210K-3.3TRG1
Connections:
- net +10V: now also C20.1, C21.1, L3.2, R28.1, U3.3 (IN)
- net +5V: now also C24.1, U3.2 (OUT); no longer C20.1, C21.1, L3.2, R28.1
- net DCDC_IN: now also C14.1, L2.1
- net GND: now also C24.2, U3.1 (GND)
Other:
- note added: "10V to 5V (LDO)"
- note added: "DCDC_IN chosen as input\nin to stay alive if solar\ngoes down for boost mode\noperation (battery on high side)"
- note added: "Place close\nto SMPS"
- note added: "Solar/Battery to 10V (SMPS)"
- note removed: "50V"
- note removed: "5V to 10V (charge pump)"
- note removed: "Battery to 5V (SMPS)"
- note removed: "Choose between PV or \nbattery as power supply\ninput (default: battery)"
- note removed: "DNP"
- moved on the sheet: C14, C15, C19, C20, C21, C23, C35, C38, C41, D2, L2, L3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

Commit message: Minor changes and gerber export update
Parts:
- C14: Comment 100V, X7S -> (none); Remarks (none) -> 100V, X7S
- C15: Comment 100V, X7R -> (none); Remarks (none) -> 100V, X7R
- C23: Remarks 25V -> 25V, X5R
- C38: Remarks (none) -> 6.3V, X5R
- D2: ALT DFLS160-7 -> (none); Alternative (none) -> DFLS160-7
- U5: ALT MIC5225 -> (none); Alternative (none) -> MIC5225
Changed lines of the file:
@@
 F 7 "" H -2200 2550 50  0001 C CNN "SPN"
 F 8 "" H -2200 2550 50  0001 C CNN "SPURL"
-F 9 "25V" H 0   0   60  0001 C CNN "Remarks"
+F 9 "25V, X5R" H 0   0   60  0001 C CNN "Remarks"
+F 10 "" H 0   0   60  0001 C CNN "Comment"
 	1    5800 5300
 	1    0    0    -1
@@
 F 4 "Diodes Inc." H 1400 200 50  0001 C CNN "Manufacturer"
 F 5 "SS16FP" H 1400 200 50  0001 C CNN "PartNumber"
-F 6 "DFLS160-7" H 6100 2800 60  0001 C CNN "ALT"
+F 6 "" H 6100 2800 60  0001 C CNN "ALT"
+F 7 "DFLS160-7" H 0   0   60  0001 C CNN "Alternative"
 	1    6100 2800
 	0    -1   1    0
@@
 F 7 "" H 1100 -50 50  0001 C CNN "SPN"
 F 8 "" H 1100 -50 50  0001 C CNN "SPURL"
-F 9 "100V, X7S" H 0   0   60  0001 C CNN "Comment"
+F 9 "" H 0   0   60  0001 C CNN "Comment"
+F 10 "100V, X7S" H 0   0   60  0001 C CNN "Remarks"
 	1    3500 2700
 	1    0    0    -1
@@
 F 4 "Murata" H 1100 -50 50  0001 C CNN "Manufacturer"
 F 5 "GRM31CR72A225KA73L" H 1100 -50 50  0001 C CNN "PartNumber"
-F 6 "100V, X7R" H 0   0   60  0001 C CNN "Comment"
+F 6 "" H 0   0   60  0001 C CNN "Comment"
 F 7 "TY HMK325B7225KN-T" H 0   0   60  0001 C CNN "Alternative"
+F 8 "100V, X7R" H 0   0   60  0001 C CNN "Remarks"
 	1    4100 2700
 	1    0    0    -1
@@
 F 7 "" H -2250 2500 50  0001 C CNN "SPN"
 F 8 "" H -2250 2500 50  0001 C CNN "SPURL"
+F 9 "" H 0   0   60  0001 C CNN "Comment"
+F 10 "6.3V, X5R" H 0   0   60  0001 C CNN "Remarks"
 	1    7500 5300
 	1    0    0    -1
@@
 F 4 "Diodes Inc." H -2250 2650 50  0001 C CNN "Manufacturer"
 F 5 "AP2210K-3.3TRG1" H -2250 2650 50  0001 C CNN "PartNumber"
-F 6 "MIC5225" H 6600 5200 60  0001 C CNN "ALT"
+F 6 "" H 6600 5200 60  0001 C CNN "ALT"
+F 7 "MIC5225" H 0   0   60  0001 C CNN "Alternative"
 	1    6600 5200
 	1    0    0    -1

Commit message: V0.8.1: Small changes and update to new kicad symbol library table (nightlies only)
Parts:
- removed C41: 100n, LibreSolar:C_0603_1608, symbol C
- C14, C19, C20, C21, C23, C24, C35, C38: symbol C -> device:C_Small
- C15: value 2.2u -> 4.7u; symbol C -> device:C_Small; Alternative TY HMK325B7225KN-T -> (none); PartNumber GRM31CR72A225KA73L -> GRJ32DC72A475KE11L; Remarks 100V, X7R -> 100V, X7S
- D2: symbol D_Schottky -> device:D_Schottky_Small
- L2, L3: symbol L -> device:L_Small
- R28, R29: symbol R -> device:R_Small
- U3: symbol AZ1117 -> LibreSolar:AZ1117
- U4: symbol LMR16006 -> LibreSolar:LMR16006
- U5: symbol AP2210-3.3 -> LibreSolar:AP2210-3.3
Changed lines of the file:
@@
-EESchema Schematic File Version 2
-LIBS:MPPT_charger_20A-rescue
-LIBS:LibreSolar
-LIBS:IEC-60617
-LIBS:power
-LIBS:device
-LIBS:regul
-LIBS:switches
-LIBS:conn
-LIBS:logo
-LIBS:mechanical
+EESchema Schematic File Version 4
 LIBS:MPPT_charger_20A-cache
 EELAYER 26 0
@@
 $EndDescr
 $Comp
-L GND #PWR036
+L power:GND #PWR036
 U 1 1 58C300D5
 P 7500 5600
@@
 $EndComp
 $Comp
-L GND #PWR037
+L power:GND #PWR037
 U 1 1 58C300DB
 P 7100 5600
@@
 $EndComp
 $Comp
-L GND #PWR038
+L power:GND #PWR038
 U 1 1 58C300E7
 P 5800 5600
@@
 $EndComp
 $Comp
-L GND #PWR039
+L power:GND #PWR039
 U 1 1 58C300ED
 P 7900 3400
@@
 $EndComp
 $Comp
-L GND #PWR040
+L power:GND #PWR040
 U 1 1 58C300F3
 P 7500 3400
@@
 $EndComp
 $Comp
-L GND #PWR041
+L power:GND #PWR041
 U 1 1 58C300F9
 P 7100 3400
@@
 $EndComp
 $Comp
-L GND #PWR042
+L power:GND #PWR042
 U 1 1 58C30100
 P 6100 3000
@@
 $EndComp
 $Comp
-L GND #PWR043
+L power:GND #PWR043
 U 1 1 58C30106
 P 4100 2900
@@
 $EndComp
 $Comp
-L GND #PWR044
+L power:GND #PWR044
 U 1 1 58C3010C
 P 4800 2900
@@
 $EndComp
 $Comp
-L GND #PWR045
+L power:GND #PWR045
 U 1 1 58C30112
 P 3500 2900
@@
 $EndComp
 $Comp
-L +3.3V #PWR046
+L power:+3.3V #PWR046
 U 1 1 58C30118
 P 7500 4900
@@
 $EndComp
 $Comp
-L R R29
+L device:R_Small R29
 U 1 1 58C3011E
 P 7100 3200
-F 0 "R29" V 7030 3200 50  0000 C CNN
-F 1 "10k" V 7170 3200 50  0000 C CNN
-F 2 "LibreSolar:R_0603_1608" H 7100 3200 50  0001 C CNN
+F 0 "R29" V 7025 3200 50  0000 C CNN
+F 1 "10k" V 7175 3200 50  0000 C CNN
+F 2 "LibreSolar:R_0603_1608" V 6925 3100 50  0001 C CNN
 F 3 "" H 7100 3200 50  0000 C CNN
 F 4 "Yageo" H 1400 200 50  0001 C CNN "Manufacturer"
@@
 $EndComp
 $Comp
-L C C23
+L device:C_Small C23
 U 1 1 58C30133
 P 5800 5300
@@
 $EndComp
 $Comp
-L C C21
+L device:C_Small C21
 U 1 1 58C3013A
 P 7900 3100
@@
 $EndComp
 $Comp
-L C C20
+L device:C_Small C20
 U 1 1 58C30141
 P 7500 3100
@@
 $EndComp
 $Comp
-L R R28
+L device:R_Small R28
 U 1 1 58C30148
 P 7100 2800
-F 0 "R28" V 7030 2800 50  0000 C CNN
-F 1 "120k" V 7170 2800 50  0000 C CNN
-F 2 "LibreSolar:R_0603_1608" H 7100 2800 50  0001 C CNN
+F 0 "R28" V 7025 2800 50  0000 C CNN
+F 1 "120k" V 7175 2800 50  0000 C CNN
+F 2 "LibreSolar:R_0603_1608" V 6925 2700 50  0001 C CNN
 F 3 "" H 7100 2800 50  0000 C CNN
 F 4 "Yageo" H 1400 200 50  0001 C CNN "Manufacturer"
@@
 $EndComp
 $Comp
-L D_Schottky D2
+L device:D_Schottky_Small D2
 U 1 1 58C3014F
 P 6100 2800
@@
 F 4 "Diodes Inc." H 1400 200 50  0001 C CNN "Manufacturer"
 F 5 "SS16FP" H 1400 200 50  0001 C CNN "PartNumber"
-F 6 "" H 6100 2800 60  0001 C CNN "ALT"
-F 7 "DFLS160-7" H 0   0   60  0001 C CNN "Alternative"
+F 6 "DFLS160-7" H 0   0   60  0001 C CNN "Alternative"
 	1    6100 2800
 	0    -1   1    0
 $EndComp
 $Comp
-L C C19
+L device:C_Small C19
 U 1 1 58C30156
 P 6050 2400
@@
 $EndComp
 $Comp
-L C C14
+L device:C_Small C14
 U 1 1 58C3015D
 P 3500 2700
@@
 $EndComp
 $Comp
-L C C15
+L device:C_Small C15
 U 1 1 58C30164
 P 4100 2700
 F 0 "C15" H 4125 2775 50  0000 L CNN
-F 1 "2.2u" H 4125 2625 50  0000 L CNN
+F 1 "4.7u" H 4125 2625 50  0000 L CNN
 F 2 "LibreSolar:C_1210_3225" H 4100 2500 50  0001 C CNN
 F 3 "" H 4125 2775 50  0000 C CNN
 F 4 "Murata" H 1100 -50 50  0001 C CNN "Manufacturer"
-F 5 "GRM31CR72A225KA73L" H 1100 -50 50  0001 C CNN "PartNumber"
-F 6 "" H 0   0   60  0001 C CNN "Comment"
-F 7 "TY HMK325B7225KN-T" H 0   0   60  0001 C CNN "Alternative"
-F 8 "100V, X7R" H 0   0   60  0001 C CNN "Remarks"
+F 5 "GRJ32DC72A475KE11L" H 1100 -50 50  0001 C CNN "PartNumber"
+F 6 "100V, X7S" H 0   0   60  0001 C CNN "Remarks"
 	1    4100 2700
 	1    0    0    -1
 $EndComp
 $Comp
-L L L2
+L device:L_Small L2
 U 1 1 58C3016B
 P 3800 2400
-F 0 "L2" H 3800 2470 50  0000 C CNN
-F 1 "4.7uH" H 3800 2350 50  0000 C CNN
+F 0 "L2" V 3870 2400 50  0000 C CNN
+F 1 "4.7uH" V 3740 2400 50  0000 C CNN
 F 2 "Inductors_SMD:L_0805" V 3800 2400 50  0001 C CNN
 F 3 "" V 3800 2400 50  0000 C CNN
 F 4 "Murata" H 1100 200 50  0001 C CNN "Manufacturer"
 F 5 "LQM21PN4R7NGRD" H 1100 200 50  0001 C CNN "PartNumber"
-F 6 "" H 1100 200 50  0001 C CNN "SPR"
-F 7 "" H 1100 200 50  0001 C CNN "SPN"
-F 8 "" H 1100 200 50  0001 C CNN "SPURL"
 	1    3800 2400
-	1    0    0    -1
-$EndComp
-$Comp
-L C C35
+	0    -1   -1   0
+$EndComp
+$Comp
+L device:C_Small C35
 U 1 1 58C3017A
 P 7100 5400
@@
 $EndComp
 $Comp
-L C C38
+L device:C_Small C38
 U 1 1 58C30181
 P 7500 5300
@@
 $EndComp
 $Comp
-L L L3
+L device:L_Small L3
 U 1 1 58C30191
 P 6650 2600
-F 0 "L3" H 6650 2670 50  0000 C CNN
-F 1 "47uH" H 6650 2550 50  0000 C CNN
+F 0 "L3" V 6720 2600 50  0000 C CNN
+F 1 "47uH" V 6590 2600 50  0000 C CNN
 F 2 "LibreSolar:L_Wuerth_WE-TPC-58xx" V 6650 2600 50  0001 C CNN
 F 3 "" V 6650 2600 50  0000 C CNN
@@
 F 6 "WE-TPC-5828 744053470" H 6650 2600 60  0001 C CNN "Alternative"
 	1    6650 2600
-	1    0    0    -1
-$EndComp
-$Comp
-L LMR16006 U4
+	0    -1   -1   0
+$EndComp
+$Comp
+L LibreSolar:LMR16006 U4
 U 1 1 58BDBD3F
 P 5300 2600
@@
 $EndComp
 $Comp
-L AP2210-3.3 U5
+L LibreSolar:AP2210-3.3 U5
 U 1 1 58BDC485
 P 6600 5200
@@
 F 4 "Diodes Inc." H -2250 2650 50  0001 C CNN "Manufacturer"
 F 5 "AP2210K-3.3TRG1" H -2250 2650 50  0001 C CNN "PartNumber"
-F 6 "" H 6600 5200 60  0001 C CNN "ALT"
-F 7 "MIC5225" H 0   0   60  0001 C CNN "Alternative"
+F 6 "MIC5225" H 0   0   60  0001 C CNN "Alternative"
 	1    6600 5200
 	1    0    0    -1
 $EndComp
 $Comp
-L GND #PWR047
+L power:GND #PWR047
 U 1 1 58BDC73F
 P 6100 5600
@@
 $EndComp
 $Comp
-L +5V #PWR048
+L power:+5V #PWR048
 U 1 1 58BDCD2C
 P 5800 4900
@@
 $EndComp
 $Comp
-L PWR_FLAG #FLG049
+L power:PWR_FLAG #FLG049
 U 1 1 58BFEDCA
-P 7600 2550
-F 0 "#FLG049" H 7600 2500 50  0001 C CNN
-F 1 "PWR_FLAG" H 7600 2750 50  0000 C CNN
-F 2 "" H 7600 2550 50  0000 C CNN
-F 3 "" H 7600 2550 50  0000 C CNN
-	1    7600 2550
-	1    0    0    -1
-$EndComp
-$Comp
-L PWR_FLAG #FLG050
+P 7600 2500
+F 0 "#FLG049" H 7600 2575 50  0001 C CNN
+F 1 "PWR_FLAG" H 7600 2650 50  0000 C CNN
+F 2 "" H 7600 2500 50  0001 C CNN
+F 3 "" H 7600 2500 50  0001 C CNN
+	1    7600 2500
+	1    0    0    -1
+$EndComp
+$Comp
+L power:PWR_FLAG #FLG050
 U 1 1 58BFEEDA
 P 4600 2300
-F 0 "#FLG050" H 4600 2250 50  0001 C CNN
-F 1 "PWR_FLAG" H 4600 2500 50  0000 C CNN
-F 2 "" H 4600 2300 50  0000 C CNN
-F 3 "" H 4600 2300 50  0000 C CNN
+F 0 "#FLG050" H 4600 2375 50  0001 C CNN
+F 1 "PWR_FLAG" H 4600 2450 50  0000 C CNN
+F 2 "" H 4600 2300 50  0001 C CNN
+F 3 "" H 4600 2300 50  0001 C CNN
 	1    4600 2300
 	1    0    0    -1
@@
 	7100 5200 7100 5300
 Wire Wire Line
-	7600 2550 7600 2600
+	7600 2500 7600 2600
 Wire Wire Line
 	4600 2300 4600 2400
@@
 Text Notes 6100 4400 0    100  ~ 0
 5V to 3.3V (LDO)
-$Comp
-L GND #PWR051
-U 1 1 58CE7EFC
-P 4400 2900
-F 0 "#PWR051" H 4400 2650 50  0001 C CNN
-F 1 "GND" H 4400 2750 50  0000 C CNN
-F 2 "" H 4400 2900 50  0000 C CNN
-F 3 "" H 4400 2900 50  0000 C CNN
-	1    4400 2900
-	1    0    0    -1
-$EndComp
-$Comp
-L C C41
-U 1 1 58CE7F0D
-P 4400 2700
-F 0 "C41" H 4425 2775 50  0000 L CNN
-F 1 "100n" H 4425 2625 50  0000 L CNN
-F 2 "LibreSolar:C_0603_1608" H 4400 2500 50  0001 C CNN
-F 3 "" H 4425 2775 50  0000 C CNN
-F 4 "Murata" H 3000 -2800 50  0001 C CNN "Manufacturer"
-F 5 "GRM188R71H104KA93D" H 3000 -2800 50  0001 C CNN "PartNumber"
-F 6 "" H 3000 -2800 50  0001 C CNN "SPR"
-F 7 "" H 3000 -2800 50  0001 C CNN "SPN"
-F 8 "" H 3000 -2800 50  0001 C CNN "SPURL"
-	1    4400 2700
-	1    0    0    -1
-$EndComp
-Wire Wire Line
-	4400 2400 4400 2600
-Wire Wire Line
-	4400 2900 4400 2800
-Connection ~ 4400 2400
 Wire Wire Line
 	5800 3200 6600 3200
@@
 	3200 2400 3700 2400
 $Comp
-L +10V #PWR052
+L LibreSolar:+10V #PWR052
 U 1 1 5911CE30
 P 7900 2500
@@
 $EndComp
 $Comp
-L AZ1117 U3
+L LibreSolar:AZ1117 U3
 U 1 1 5911D439
 P 3300 5300
@@
 $EndComp
 $Comp
-L GND #PWR053
+L power:GND #PWR053
 U 1 1 5911D540
 P 2800 5700
@@
 $EndComp
 $Comp
-L C C24
+L device:C_Small C24
 U 1 1 5911D658
 P 3900 5400
@@
 $EndComp
 $Comp
-L GND #PWR054
+L power:GND #PWR054
 U 1 1 5911D778
 P 3900 5700
@@
 	3900 5000 3900 5300
 $Comp
-L +5V #PWR055
+L power:+5V #PWR055
 U 1 1 5911D9AC
 P 3900 5000
@@
 DCDC_IN chosen as input\nin to stay alive if solar\ngoes down for boost mode\noperation (battery on high side)
 $Comp
-L +10V #PWR056
+L LibreSolar:+10V #PWR056
 U 1 1 59569E56
 P 2800 5000
