File: analog_frontend.sch (KiCad schematic (older format))
At the start: 26 parts, among them U7 LM358

Commit message: V0.8.1: Small changes and update to new kicad symbol library table (nightlies only)
Parts:
- removed U7: LM358, Housings_SOIC:SOIC-8_3.9x4.9mm_Pitch1.27mm, symbol LM358
- added U7: LM258, LibreSolar:SOIC-8_3.9x4.9mm_Pitch1.27mm, symbol device:Opamp_Dual_Generic
- C11, C13, C16, C17, C18, C40, C42, C9: symbol C -> device:C_Small
- R11, R14, R15, R18, R19, R20, R21, R22, R23, R24, R25, R26, R27, R44, R7, R8: symbol R -> device:R_Small
- RT1: symbol Thermistor_NTC -> IEC-60617:Thermistor_NTC
Connections:
- net +5V: now also U7.8 (V+)
- net GND: now also U7.4 (V-)
- net at R15.1, R7.1: now also U7.6 (-)
- net at R14.2, R8.1: now also U7.5 (+)
- net at R11.1, R15.2: now also U7.7
- net at R20.1, R22.2: now also U7.1
- net at R18.1, R22.1: now also U7.2 (-)
- net at R19.1, R21.1: now also U7.3 (+)
Other:
- moved on the sheet: C11, C13, C42, R11, R14, R15, R18, R19, R20, R21, R22, R7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

Commit message: Revision 0.9 for first small production batch - Switchable power supply for bus and UEXT (to be make sure to reach very low power consumption during LVD conditions) - MLCCs for EMC added to each high power input/output - Re-arrangement of some connectors after initial tests with housing
Parts:
- C11, C13, C17, C18: value 100n -> 10n; PartNumber GRM188R71H104KA93D -> GRM188R71H103KA01D
- R11, R20: value 1k -> 2.2k; PartNumber RC0603FR-071KL -> RC0603FR-072K2L
- R23, R27, R44: PartNumber RC0603FR-07150KL -> RC0603FR-0710KL
Other:
- moved on the sheet: C16, C40, R23, R24, R25, R44, RT1

Commit message: Final version for Jan/2018 production
Parts:
- C11, C13, C17, C18: PartNumber GRM188R71H103KA01D -> GRM188R71H103KA01J
Changed lines of the file:
@@
 Sheet 6 6
 Title "MPPT Charger 20A"
-Date "2017-12-11"
-Rev "0.9"
+Date "2018-01-18"
+Rev "0.10"
 Comp "Libre Solar"
 Comment1 "Author: Martin Jäger"
@@
 F 3 "" H 8025 5675 50  0000 C CNN
 F 4 "Murata" H 700 -200 50  0001 C CNN "Manufacturer"
-F 5 "GRM188R71H103KA01D" H 700 -200 50  0001 C CNN "PartNumber"
+F 5 "GRM188R71H103KA01J" H 700 -200 50  0001 C CNN "PartNumber"
 	1    8000 5600
 	1    0    0    -1
@@
 F 3 "" H 6825 5675 50  0000 C CNN
 F 4 "Murata" H 650 -200 50  0001 C CNN "Manufacturer"
-F 5 "GRM188R71H103KA01D" H 650 -200 50  0001 C CNN "PartNumber"
+F 5 "GRM188R71H103KA01J" H 650 -200 50  0001 C CNN "PartNumber"
 	1    6800 5600
 	1    0    0    -1
@@
 F 3 "" H 9700 2600 50  0001 C CNN
 F 4 "Murata" H -650 -1600 50  0001 C CNN "Manufacturer"
-F 5 "GRM188R71H103KA01D" H -650 -1600 50  0001 C CNN "PartNumber"
+F 5 "GRM188R71H103KA01J" H -650 -1600 50  0001 C CNN "PartNumber"
 	1    9700 2600
 	1    0    0    -1
@@
 F 3 "" H 5700 2600 50  0000 C CNN
 F 4 "Murata" H 1950 -4500 50  0001 C CNN "Manufacturer"
-F 5 "GRM188R71H103KA01D" H 1950 -4500 50  0001 C CNN "PartNumber"
+F 5 "GRM188R71H103KA01J" H 1950 -4500 50  0001 C CNN "PartNumber"
 	1    5700 2600
 	1    0    0    -1

Commit message: Update to KiCad 5 schematic library
Parts:
- C11, C13, C16, C17, C18, C40, C42, C9: symbol device:C_Small -> Project:C
- R11, R14, R15, R18, R19, R20, R21, R22, R23, R24, R25, R26, R27, R44, R7, R8: symbol device:R_Small -> Project:R
- RT1: symbol IEC-60617:Thermistor_NTC -> Device:Thermistor_NTC
- U7: symbol device:Opamp_Dual_Generic -> Device:Opamp_Dual_Generic
Changed lines of the file:
@@
 $EndComp
 $Comp
-L device:R_Small R27
+L Project:R R27
 U 1 1 58A6E7F1
 P 8400 5600
@@
 $EndComp
 $Comp
-L device:R_Small R25
+L Project:R R25
 U 1 1 58A70DA1
 P 8400 5000
@@
 $EndComp
 $Comp
-L device:R_Small R24
+L Project:R R24
 U 1 1 58A715AF
 P 7200 5000
@@
 $EndComp
 $Comp
-L device:R_Small R26
+L Project:R R26
 U 1 1 58A71DE2
 P 7200 5600
@@
 $EndComp
 $Comp
-L device:C_Small C18
+L Project:C C18
 U 1 1 58A723ED
 P 8000 5600
@@
 $EndComp
 $Comp
-L device:C_Small C17
+L Project:C C17
 U 1 1 58A72885
 P 6800 5600
@@
 $EndComp
 $Comp
-L device:C_Small C16
+L Project:C C16
 U 1 1 58A7377B
 P 2200 5500
@@
 $EndComp
 $Comp
-L device:R_Small R23
+L Project:R R23
 U 1 1 58A7452B
 P 2700 4900
@@
 $EndComp
 $Comp
-L IEC-60617:Thermistor_NTC RT1
+L Device:Thermistor_NTC RT1
 U 1 1 58A75726
 P 2700 5500
@@
 $EndComp
 $Comp
-L device:C_Small C13
+L Project:C C13
 U 1 1 58A7ED33
 P 9700 2600
@@
 $EndComp
 $Comp
-L device:C_Small C9
+L Project:C C9
 U 1 1 58A847D1
 P 2300 2400
@@
 $EndComp
 $Comp
-L device:C_Small C11
+L Project:C C11
 U 1 1 58A86B85
 P 5700 2600
@@
 $EndComp
 $Comp
-L device:R_Small R7
+L Project:R R7
 U 1 1 58A9F3FF
 P 4100 2400
@@
 $EndComp
 $Comp
-L device:R_Small R8
+L Project:R R8
 U 1 1 58A9F8B2
 P 3900 2200
@@
 $EndComp
 $Comp
-L device:R_Small R11
+L Project:R R11
 U 1 1 58AA2C36
 P 5500 2300
@@
 $EndComp
 $Comp
-L device:R_Small R15
+L Project:R R15
 U 1 1 58AA3509
 P 5000 2900
@@
 $EndComp
 $Comp
-L device:R_Small R14
+L Project:R R14
 U 1 1 58AA3A32
 P 4100 1900
@@
 $EndComp
 $Comp
-L device:R_Small R19
+L Project:R R19
 U 1 1 58AA826A
 P 8000 2200
@@
 $EndComp
 $Comp
-L device:R_Small R18
+L Project:R R18
 U 1 1 58AA8A90
 P 8200 2400
@@
 $EndComp
 $Comp
-L device:R_Small R22
+L Project:R R22
 U 1 1 58AAB023
 P 8900 2800
@@
 $EndComp
 $Comp
-L device:R_Small R21
+L Project:R R21
 U 1 1 58AAB89C
 P 8200 1900
@@
 $EndComp
 $Comp
-L device:R_Small R20
+L Project:R R20
 U 1 1 58AACEAA
 P 9500 2300
@@
 $EndComp
 $Comp
-L device:C_Small C40
+L Project:C C40
 U 1 1 58CBE39F
 P 3500 5550
@@
 $EndComp
 $Comp
-L device:R_Small R44
+L Project:R R44
 U 1 1 58CBE7D6
 P 3500 4900
@@
 	2200 5600 2200 5800
 Wire Wire Line
-	2700 5600 2700 5800
-Wire Wire Line
-	9600 2300 9850 2300
+	2700 5650 2700 5800
+Wire Wire Line
+	9600 2300 9700 2300
 Wire Wire Line
 	9700 2300 9700 2500
 Wire Wire Line
-	5600 2300 5900 2300
+	5600 2300 5700 2300
 Wire Wire Line
 	5700 2300 5700 2500
@@
 	9300 2800 9300 2300
 Wire Wire Line
-	9200 2300 9400 2300
-Wire Wire Line
-	8100 2200 8600 2200
+	9200 2300 9300 2300
+Wire Wire Line
+	8100 2200 8500 2200
 Wire Wire Line
 	8500 2200 8500 1900
 Wire Wire Line
-	4000 2200 4500 2200
+	4000 2200 4400 2200
 Wire Wire Line
 	4400 2200 4400 1900
 Wire Wire Line
-	8300 2400 8600 2400
+	8300 2400 8500 2400
 Wire Wire Line
 	8500 2400 8500 2800
@@
 	8500 2800 8800 2800
 Wire Wire Line
-	5100 2300 5400 2300
+	5100 2300 5300 2300
 Wire Wire Line
 	5100 2900 5300 2900
@@
 	5300 2900 5300 2300
 Wire Wire Line
-	4200 2400 4500 2400
+	4200 2400 4400 2400
 Wire Wire Line
 	4900 2900 4400 2900
@@
 	2200 5400 2200 5200
 Wire Wire Line
-	2200 5200 2800 5200
-Wire Wire Line
-	2700 5000 2700 5400
+	2200 5200 2700 5200
+Wire Wire Line
+	2700 5000 2700 5200
 Wire Wire Line
 	8000 5300 8000 5500
 Wire Wire Line
-	8000 5300 8500 5300
-Wire Wire Line
-	8400 5100 8400 5500
+	8000 5300 8400 5300
+Wire Wire Line
+	8400 5100 8400 5300
 Wire Wire Line
 	6800 5300 6800 5500
 Wire Wire Line
-	6800 5300 7300 5300
-Wire Wire Line
-	7200 5100 7200 5500
+	6800 5300 7200 5300
+Wire Wire Line
+	7200 5100 7200 5300
 Wire Wire Line
 	3500 4700 3500 4800
 Wire Wire Line
-	3500 5000 3500 5450
+	3500 5000 3500 5200
 Wire Wire Line
 	3500 5200 3900 5200
@@
 Connection ~ 3500 5200
 $Comp
-L device:C_Small C42
+L Project:C C42
 U 1 1 58CE9BFF
 P 1400 2400
@@
 	2300 2000 2700 2000
 Wire Wire Line
-	2700 1900 2700 2100
+	2700 1900 2700 2000
 Connection ~ 2700 2000
 Wire Wire Line
-	2700 2700 2700 2900
+	2700 2700 2700 2800
 Wire Wire Line
 	2700 2800 2300 2800
@@
 Connection ~ 2700 2800
 $Comp
-L device:Opamp_Dual_Generic U7
+L Device:Opamp_Dual_Generic U7
 U 1 1 5A1ADFEF
 P 8900 2300
@@
 $EndComp
 $Comp
-L device:Opamp_Dual_Generic U7
+L Device:Opamp_Dual_Generic U7
 U 2 1 5A1AE438
 P 4800 2300
@@
 $EndComp
 $Comp
-L device:Opamp_Dual_Generic U7
+L Device:Opamp_Dual_Generic U7
 U 3 1 5A1AE618
 P 2800 2400
@@
 	1    0    0    -1
 $EndComp
+Wire Wire Line
+	9700 2300 9850 2300
+Wire Wire Line
+	5700 2300 5900 2300
+Wire Wire Line
+	9300 2300 9400 2300
+Wire Wire Line
+	8500 2200 8600 2200
+Wire Wire Line
+	4400 2200 4500 2200
+Wire Wire Line
+	8500 2400 8600 2400
+Wire Wire Line
+	5300 2300 5400 2300
+Wire Wire Line
+	4400 2400 4500 2400
+Wire Wire Line
+	2700 5200 2800 5200
+Wire Wire Line
+	2700 5200 2700 5350
+Wire Wire Line
+	8400 5300 8500 5300
+Wire Wire Line
+	8400 5300 8400 5500
+Wire Wire Line
+	7200 5300 7300 5300
+Wire Wire Line
+	7200 5300 7200 5500
+Wire Wire Line
+	3500 5200 3500 5450
+Wire Wire Line
+	2700 2000 2700 2100
+Wire Wire Line
+	2700 2800 2700 2900
 $EndSCHEMATC
