File: dcdc.sch (KiCad schematic (older format))
At the start: 61 parts, among them J1 SOLAR, J2 LOAD, J3 BAT, J5 TEMP, Q1 CSD18540Q5B, Q2 CSD18540Q5B, Q3 CSD18540Q5B, Q4 CSD18540Q5B, T1 MMBT3904, U1 LM5107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

Commit message: Updated R/C/L symbols to IEC 60617 style
Parts:
- C1, C2: Comment (none) -> 63V, 2.74A, 16x25
- C3: Comment (none) -> 100V, X7R
- C4: Comment (none) -> 100V, X7S
- C5: Comment (none) -> 100V
- D1: symbol D_ALT -> D
- RT1: renamed from NTC1; value 10k-NTC -> 10k
Other:
- note added: "Temperature (ext./int.)"
- note removed: "1000uF, 63V, 2.73A, 16x25\nUnited Chemi EKYB630ELL102ML25S"
- note removed: "1u, 100V, X7S\nTDK C2012X7S2A105M125AB\n2.2u, 100V, X7R\nMurata GRM31CR72A225KA73L"
- moved on the sheet: C1, C10, C11, C12, C13, C16, C17, C18, C2, C3, C4, C40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

Commit message: Updated revision: 0.8
Parts:
- removed C11, C13, C16, C17, C18, C40, C42, C9: 100n, Capacitors_SMD:C_0603, symbol C
- removed C7, C8: 820u, Capacitors_THT:C_Radial_D10_L25_P5, symbol CP
- removed J5: TEMP, Connectors_Terminal_Blocks:TerminalBlock_Pheonix_MKDS1.5-2pol, symbol Screw_Terminal_1x02
- removed R11, R20: 1k, Resistors_SMD:R_0603, symbol R
- removed R14, R15, R21, R22: 150k, Resistors_SMD:R_0603, symbol R
- removed R18, R19, R7, R8: 2.2k, Resistors_SMD:R_0603, symbol R
- removed R23, R27, R44: 10k, Resistors_SMD:R_0603, symbol R
- removed R24, R25: 100k, Resistors_SMD:R_0603, symbol R
- removed R26: 5.6k, Resistors_SMD:R_0603, symbol R
- removed RT1: 10k, Resistors_SMD:R_0603, symbol Thermistor_NTC
- removed U7: LM358, Housings_SOIC:SOIC-8_3.9x4.9mm_Pitch1.27mm, symbol LM358
- added C1: 1000u, Capacitors_THT:CP_Radial_D16.0mm_P7.50mm, symbol CP
- added HS1: Heatsink_PAD, LibreSolar:Fischer_Elektronik_FK_250_10_LF_PAK, symbol Heatsink_PAD
- C10: footprint Capacitors_SMD:C_0603 -> LibreSolar:C_0603_1608; MFR Murata -> (none); MPN GRM188R71H104KA93D -> (none); Manufacturer (none) -> Murata; PartNumber (none) -> GRM188R71H104KA93D
- C12: footprint Capacitors_SMD:C_0603 -> LibreSolar:C_0603_1608; MFR Murata -> (none); MPN GRM188R61E105KA12D -> (none); Manufacturer (none) -> Murata; PartNumber (none) -> GRM188R61E105KA12D; Remarks (none) -> 25V
- C2: renamed from C1; MFR United Chemi-Con -> (none); MPN EKYB630ELL102ML25S -> (none); Manufacturer (none) -> United Chemi-Con; PartNumber (none) -> EKYB630ELL102ML25S
- C3: footprint Capacitors_SMD:C_1206 -> LibreSolar:C_1210_3225; Alternative (none) -> TY HMK325B7225KN-T; MFR Murata -> (none); MPN GRM31CR72A225KA73L -> (none); Manufacturer (none) -> Murata; PartNumber (none) -> GRM31CR72A225KA73L
- C4: footprint Capacitors_SMD:C_0805 -> LibreSolar:C_0805_2012; MFR Murata -> (none); MPN GRJ21BC72A105KE11L -> (none); Manufacturer (none) -> Murata; PartNumber (none) -> GRJ21BC72A105KE11L
- C5: renamed from C2; value 1000u -> 820u; footprint Capacitors_THT:CP_Radial_D16.0mm_P7.50mm -> Capacitors_THT:CP_Radial_D10.0mm_P5.00mm; Comment 63V, 2.74A, 16x25 -> 35V, 2.47A; MFR United Chemi-Con -> (none); MPN EKYB630ELL102ML25S -> (none); Manufacturer (none) -> Panasonic; PartNumber (none) -> EEU-FR1V821L; Voltage (none) -> 35V
- C6: footprint Capacitors_SMD:C_0805 -> LibreSolar:C_0603_1608; MFR Murata -> (none); MPN GRM1885C2A102JA01D -> (none); Manufacturer (none) -> Murata; PartNumber (none) -> GRM1885C2A102JA01D; Remarks (none) -> NP0/C0G
- C8: renamed from C5; footprint Capacitors_SMD:C_0805 -> LibreSolar:C_0805_2012; Comment 100V -> 100V, X7S; MFR Murata -> (none); MPN GRJ21BC72A105KE11L -> (none); Manufacturer (none) -> Murata; PartNumber (none) -> GRJ21BC72A105KE11L
- D1: value 1N4148W-7-F -> 1N4148; footprint Diodes_SMD:D_SOD-123 -> LibreSolar:D_SOD-123; MFR Diodes Inc. -> (none); MPN 1N4148W-7-F -> (none); Manufacturer (none) -> Diodes Inc.; PartNumber (none) -> 1N4148W-7-F; SPR Mouser -> (none)
- F1: MFR Keystone -> (none); MPN 3557-2 -> (none); Manufacturer (none) -> Keystone; PartNumber (none) -> 3557-2
- J1, J2, J3: footprint LibreSolar:MKDS_5-2-952 -> LibreSolar:Phoenix_Contact_MKDS_5-2-952; Field4 SMKDS_5/2-9,52 -> (none); MFR Phoenix Contact -> (none); MPN MKDS 5/ 2-9,5 -> (none); Manufacturer (none) -> Phoenix Contact; PartNumber (none) -> 1868076; SPN 1714971 -> (none); SPR Phoenix Contact -> (none)
- L1: MFR Feryster -> (none); MPN DTMSS-27/0,033/20-H -> (none); Manufacturer (none) -> Feryster; PartNumber (none) -> DTMSS-27/0,033/20-H
- Q1, Q2, Q3, Q4: MFR Texas Instruments -> (none); MPN CSD18540Q5BT -> (none); Manufacturer (none) -> Texas Instruments; PartNumber (none) -> CSD18540Q5BT
- R1, R10, R3: footprint Resistors_SMD:R_0805 -> LibreSolar:R_0805_2012; MFR Yageo -> (none); MPN RC0805FR-073R3L -> (none); Manufacturer (none) -> Yageo; PartNumber (none) -> RC0805FR-073R3L
- R12, R13: footprint Resistors_SMD:R_0603 -> LibreSolar:R_0603_1608; MFR Yageo -> (none); MPN RC0603FR-072K2L -> (none); Manufacturer (none) -> Yageo; PartNumber (none) -> RC0603FR-072K2L
- R16: footprint Resistors_SMD:R_0603 -> LibreSolar:R_0603_1608; MFR Yageo -> (none); MPN RC0603FR-07150KL -> (none); Manufacturer (none) -> Yageo; PartNumber (none) -> RC0603FR-07150KL
- R17, R6: MFR Bourns -> (none); MPN CRE2512-FZ-R002E-3 -> (none); Manufacturer (none) -> Bourns; PartNumber (none) -> CRE2512-FZ-R002E-3
- R2: footprint Resistors_SMD:R_0603 -> LibreSolar:R_0603_1608; MFR Yageo -> (none); MPN RC0603FR-071ML -> (none); Manufacturer (none) -> Yageo; PartNumber (none) -> RC0603FR-071ML
- R4, R5: footprint Resistors_SMD:R_1206 -> LibreSolar:R_1206_3216; MFR Yageo -> (none); MPN RC1206FR-074R7L -> (none); Manufacturer (none) -> Yageo; PartNumber (none) -> RC1206FR-074R7L
- R9: value 33k -> 56k; footprint Resistors_SMD:R_0603 -> LibreSolar:R_0603_1608; MFR Yageo -> (none); MPN RC0603FR-0733KL -> (none); Manufacturer (none) -> Yageo; PartNumber (none) -> RC0603FR-0756KL
- T1: footprint TO_SOT_Packages_SMD:SOT-23 -> LibreSolar:SOT-23; MFR Diodes Inc. -> (none); MPN MMBT3904-7-F -> (none); Manufacturer (none) -> Diodes Inc.; PartNumber (none) -> MMBT3904-7-F
- U1: MFR Texas Instruments -> (none); MPN LM5107MA -> (none); Manufacturer (none) -> Texas Instruments; PartNumber (none) -> LM5107MA
Connections:
- net BAT+: now also F1.2
- net DCDC_IN: now also C1.1, HS1.1; no longer C5.1
- net DCDC_OUT: now also C5.1, F1.1, J2.1; no longer J2.2
- net GND: now also C1.2
- net LOAD-: now also J2.2; no longer J2.1
- net LOAD-GND renamed LOAD-SW
Other:
- note removed: "25V"
- note removed: "820u, 35V, 2.47A\nPanasonic EEU-FR1V821L"
- note removed: "DCDC current"
- note removed: "Diff. amp. reference\ndefined by DAC pin\ninstead of GND: variable\nzero current set point"
- note removed: "NP0/C0G\ntype cap."
- note removed: "Solar and battery voltage"
- note removed: "Temperature (ext./int.)"
- moved on the sheet: C10, C12, C2, C3, C4, C5, C6, C8, D1, F1, J1, J2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

Commit message: Minor changes and gerber export update
Parts:
- C1, C2: Comment 63V, 2.74A, 16x25 -> (none); Remarks (none) -> 63V, 2.74A, 16x25
- C12: Remarks 25V -> 25V, X5R
- C3: Comment 100V, X7R -> (none); Remarks (none) -> 100V, X7R
- C4, C8: Comment 100V, X7S -> (none); Remarks (none) -> 100V, X7S
- C5: Comment 35V, 2.47A -> (none); Remarks (none) -> 35V, 2.47A; Voltage 35V -> (none)
- J1, J2, J3: PartNumber 1868076 -> 1714971
Changed lines of the file:
@@
 F 4 "Murata" H 500 350 50  0001 C CNN "Manufacturer"
 F 5 "GRJ21BC72A105KE11L" H 500 350 50  0001 C CNN "PartNumber"
-F 6 "100V, X7S" H 500 350 50  0001 C CNN "Comment"
+F 6 "" H 500 350 50  0001 C CNN "Comment"
+F 7 "100V, X7S" H 0   0   60  0001 C CNN "Remarks"
 	1    2600 2100
 	1    0    0    -1
@@
 F 4 "Murata" H 100 300 50  0001 C CNN "Manufacturer"
 F 5 "GRJ21BC72A105KE11L" H 100 300 50  0001 C CNN "PartNumber"
-F 6 "100V, X7S" H 100 300 50  0001 C CNN "Comment"
+F 6 "" H 100 300 50  0001 C CNN "Comment"
+F 7 "100V, X7S" H 0   0   60  0001 C CNN "Remarks"
 	1    4700 2100
 	1    0    0    -1
@@
 F 4 "Murata" H -800 950 50  0001 C CNN "Manufacturer"
 F 5 "GRM188R61E105KA12D" H -800 950 50  0001 C CNN "PartNumber"
-F 6 "25V" H 2250 5000 50  0000 C CNN "Remarks"
+F 6 "25V, X5R" H 2250 5000 50  0000 C CNN "Remarks"
+F 7 "" H 0   0   60  0001 C CNN "Comment"
 	1    2400 5000
 	1    0    0    -1
@@
 F 3 "" H 9975 2800 50  0001 C CNN
 F 4 "Phoenix Contact" H 0   0   60  0001 C CNN "Manufacturer"
-F 5 "1868076" H 0   0   60  0001 C CNN "PartNumber"
+F 5 "1714971" H 0   0   60  0001 C CNN "PartNumber"
 	1    10000 2800
 	-1   0    0    1
@@
 F 3 "" H 1625 2100 50  0001 C CNN
 F 4 "Phoenix Contact" H 1650 2100 60  0001 C CNN "Manufacturer"
-F 5 "1868076" H 1650 2100 60  0001 C CNN "PartNumber"
+F 5 "1714971" H 1650 2100 60  0001 C CNN "PartNumber"
 	1    1650 2100
 	1    0    0    1
@@
 F 3 "" H 9875 5400 50  0001 C CNN
 F 4 "Phoenix Contact" H 0   0   60  0001 C CNN "Manufacturer"
-F 5 "1868076" H 0   0   60  0001 C CNN "PartNumber"
+F 5 "1714971" H 0   0   60  0001 C CNN "PartNumber"
 	1    9900 5400
 	-1   0    0    -1
@@
 F 4 "United Chemi-Con" H 600 300 50  0001 C CNN "Manufacturer"
 F 5 "EKYB630ELL102ML25S" H 600 300 50  0001 C CNN "PartNumber"
-F 6 "63V, 2.74A, 16x25" H 4025 1925 50  0001 L CNN "Comment"
+F 6 "" H 4025 1925 50  0001 L CNN "Comment"
+F 7 "63V, 2.74A, 16x25" H 0   0   60  0001 C CNN "Remarks"
 	1    4000 2100
 	1    0    0    -1
@@
 F 4 "Panasonic" H 4200 1000 50  0001 C CNN "Manufacturer"
 F 5 "EEU-FR1V821L" H 4200 1000 50  0001 C CNN "PartNumber"
-F 6 "35V, 2.47A" H 8000 2800 60  0001 C CNN "Comment"
-F 7 "35V" H 8020 2650 50  0000 L CNN "Voltage"
+F 6 "35V, 2.47A" H 0   0   60  0001 C CNN "Remarks"
 	1    8000 2800
 	1    0    0    -1
@@
 F 4 "Murata" H 200 300 50  0001 C CNN "Manufacturer"
 F 5 "GRM31CR72A225KA73L" H 200 300 50  0001 C CNN "PartNumber"
-F 6 "100V, X7R" H 4400 2100 60  0001 C CNN "Comment"
+F 6 "" H 4400 2100 60  0001 C CNN "Comment"
 F 7 "TY HMK325B7225KN-T" H 0   0   60  0001 C CNN "Alternative"
+F 8 "100V, X7R" H 0   0   60  0001 C CNN "Remarks"
 	1    4400 2100
 	1    0    0    -1
@@
 F 4 "United Chemi-Con" H 200 300 50  0001 C CNN "Manufacturer"
 F 5 "EKYB630ELL102ML25S" H 200 300 50  0001 C CNN "PartNumber"
-F 6 "63V, 2.74A, 16x25" H 3625 1925 50  0001 L CNN "Comment"
+F 6 "" H 3625 1925 50  0001 L CNN "Comment"
+F 7 "63V, 2.74A, 16x25" H 0   0   60  0001 C CNN "Remarks"
 	1    3600 2100
 	1    0    0    -1

Commit message: V0.8.1: Small changes and update to new kicad symbol library table (nightlies only)
Parts:
- removed HS1: Heatsink_PAD, LibreSolar:Fischer_Elektronik_FK_250_10_LF_PAK, symbol Heatsink_PAD
- removed R5: 4.7, LibreSolar:R_1206_3216, symbol R
- C1, C2, C5: symbol CP -> device:CP_Small
- C10, C12, C6, C8: symbol C -> device:C_Small
- C3: value 2.2u -> 4.7u; symbol C -> device:C_Small; Alternative TY HMK325B7225KN-T -> (none); PartNumber GRM31CR72A225KA73L -> GRJ32DC72A475KE11L; Remarks 100V, X7R -> 100V, X7S
- C4: value 1u -> 4.7u; footprint LibreSolar:C_0805_2012 -> LibreSolar:C_1210_3225; symbol C -> device:C_Small; PartNumber GRJ21BC72A105KE11L -> GRJ32DC72A475KE11L
- D1: symbol D -> device:D_Small
- F1: symbol Fuse -> device:Fuse_Small
- J1, J2, J3: symbol Screw_Terminal_1x02 -> LibreSolar:Screw_Terminal_1x02
- L1: symbol L_Core_Iron -> device:L_Core_Iron; PartNumber DTMSS-27/0,033/20-H -> DTMSS-27/0,022/30-H
- Q1, Q2, Q3, Q4: symbol Q_NMOS -> LibreSolar:Q_NMOS
- R1, R10, R12, R13, R16, R17, R2, R3, R6, R9: symbol R -> device:R_Small
- R4: value 4.7 -> 2.2; symbol R -> device:R_Small; PartNumber RC1206FR-074R7L -> RC1206FR-072R2L
- T1: symbol MMBT3904 -> Transistor:BC817
- U1: footprint Housings_SOIC:SOIC-8_3.9x4.9mm_Pitch1.27mm -> LibreSolar:SOIC-8_3.9x4.9mm_Pitch1.27mm; symbol LM5107 -> LibreSolar:LM5107
Other:
- moved on the sheet: C6, R4

Commit message: Revision 0.9 for first small production batch - Switchable power supply for bus and UEXT (to be make sure to reach very low power consumption during LVD conditions) - MLCCs for EMC added to each high power input/output - Re-arrangement of some connectors after initial tests with housing
Parts:
- added C27, C7: 1u, LibreSolar:C_0805_2012, symbol device:C_Small
- added C28: 10n, LibreSolar:C_0603_1608, symbol device:C_Small
- added D5: SMBJ36A, LibreSolar:D_SMB, symbol device:D_Zener_Small
- C12: footprint LibreSolar:C_0603_1608 -> LibreSolar:C_0805_2012; PartNumber GRM188R61E105KA12D -> GRJ21BR71H105KE01; Remarks 25V, X5R -> (none)
- L1: SPR Feryster -> (none); Supplier (none) -> Feryster
- R16: PartNumber RC0603FR-07150KL -> RC0603FR-0710KL
- R17, R6: SPR Mouser -> (none)
Connections:
- net BAT+: now also C7.1
- net BAT-: now also C7.2
- net DCDC_OUT: now also C27.1, D5.1 (K)
- net LOAD-: now also C27.2, C28.2, D5.2 (A)
- net at Q3.G, R12.1: now also C28.1
Other:
- moved on the sheet: C10, C12, J2, Q3, R10, R12, R13, R16, R17, R9, T1, U1

Commit message: Final version for Jan/2018 production
Parts:
- C12: value 1u -> 2.2u; footprint LibreSolar:C_0805_2012 -> LibreSolar:C_0603_1608; PartNumber GRJ21BR71H105KE01 -> GRM188R61E225KA12D; Remarks (none) -> 25V, X5R
- C27, C7: PartNumber GRJ21BR71H105KE01 -> GRJ21BC72A105KE11L; Remarks (none) -> 100V, X7S
- C28: PartNumber GRM188R71H103KA01D -> GRM188R71H103KA01J
- U1: PartNumber LM5107MA -> LM5107MAX/NOPB
Changed lines of the file:
@@
 Sheet 2 6
 Title "MPPT Charger 20A"
-Date "2017-12-11"
-Rev "0.9"
+Date "2018-01-18"
+Rev "0.10"
 Comp "Libre Solar"
 Comment1 "Author: Martin Jäger"
@@
 P 7900 5200
 F 0 "C12" H 7920 5270 50  0000 L CNN
-F 1 "1u" H 7920 5130 50  0000 L CNN
-F 2 "LibreSolar:C_0805_2012" H 7900 5200 50  0001 C CNN
+F 1 "2.2u" H 7920 5130 50  0000 L CNN
+F 2 "LibreSolar:C_0603_1608" H 7900 5200 50  0001 C CNN
 F 3 "" H 7900 5200 50  0000 C CNN
 F 4 "Murata" H 4700 1150 50  0001 C CNN "Manufacturer"
-F 5 "GRJ21BR71H105KE01" H 4700 1150 50  0001 C CNN "PartNumber"
-F 6 "" H 7600 5200 50  0000 C CNN "Remarks"
+F 5 "GRM188R61E225KA12D" H 0   0   60  0001 C CNN "PartNumber"
+F 6 "25V, X5R" H 0   0   60  0001 C CNN "Remarks"
 	1    7900 5200
 	1    0    0    -1
@@
 F 3 "" H 8950 5200 60  0001 C CNN
 F 4 "Texas Instruments" H 4700 1150 50  0001 C CNN "Manufacturer"
-F 5 "LM5107MA" H 4700 1150 50  0001 C CNN "PartNumber"
+F 5 "LM5107MAX/NOPB" H 4700 1150 50  0001 C CNN "PartNumber"
 	1    8900 5200
 	1    0    0    -1
@@
 F 3 "" H 9400 2800 50  0000 C CNN
 F 4 "Murata" H 7300 1050 50  0001 C CNN "Manufacturer"
-F 5 "GRJ21BR71H105KE01" H 7300 1050 50  0001 C CNN "PartNumber"
+F 5 "GRJ21BC72A105KE11L" H 7300 1050 50  0001 C CNN "PartNumber"
+F 6 "100V, X7S" H 0   0   60  0001 C CNN "Remarks"
 	1    9400 2800
 	1    0    0    -1
@@
 F 3 "" H 5700 5700 50  0000 C CNN
 F 4 "Murata" H 3600 3950 50  0001 C CNN "Manufacturer"
-F 5 "GRJ21BR71H105KE01" H 3600 3950 50  0001 C CNN "PartNumber"
+F 5 "GRJ21BC72A105KE11L" H 3600 3950 50  0001 C CNN "PartNumber"
+F 6 "100V, X7S" H 0   0   60  0001 C CNN "Remarks"
 	1    5700 5700
 	1    0    0    -1
@@
 F 3 "" H 4100 5600 50  0000 C CNN
 F 4 "Murata" H 2000 3850 50  0001 C CNN "Manufacturer"
-F 5 "GRM188R71H103KA01D" H 2000 3850 50  0001 C CNN "PartNumber"
+F 5 "GRM188R71H103KA01J" H 2000 3850 50  0001 C CNN "PartNumber"
 	1    4100 5600
 	1    0    0    -1
