File: dcdc.sch (KiCad schematic (older format))
At the start: 36 parts, among them J1 SOLAR, J2 LOAD, J3 BAT, Q1 CSD18540Q5B, Q2 CSD18540Q5B, Q3 CSD18540Q5B, Q4 CSD18540Q5B, T1 MMBT3904, U1 LM5107

Commit message: Update to KiCad 5 schematic library
Parts:
- C1, C2: footprint Capacitors_THT:CP_Radial_D16.0mm_P7.50mm -> Capacitor_THT:CP_Radial_D16.0mm_P7.50mm; symbol device:CP_Small -> Device:CP_Small
- C10, C12, C27, C28, C3, C4, C6, C7, C8: symbol device:C_Small -> Project:C
- C5: footprint Capacitors_THT:CP_Radial_D10.0mm_P5.00mm -> Capacitor_THT:CP_Radial_D10.0mm_P5.00mm; symbol device:CP_Small -> Device:CP_Small
- D1: symbol device:D_Small -> Project:D
- D5: symbol device:D_Zener_Small -> Device:D_Zener_Small
- F1: symbol device:Fuse_Small -> Device:Fuse_Small
- J1, J2, J3: symbol LibreSolar:Screw_Terminal_1x02 -> Project:Screw_Terminal_1x02
- L1: symbol device:L_Core_Iron -> Device:L_Core_Iron
- Q1, Q2, Q3, Q4: symbol LibreSolar:Q_NMOS -> Project:Q_NMOS
- R1, R10, R12, R13, R16, R17, R2, R3, R4, R6, R9: symbol device:R_Small -> Project:R
- T1: symbol Transistor:BC817 -> Transistor_BJT:BC817
- U1: symbol LibreSolar:LM5107 -> Project:LM5107
Other:
- note added: "typisch: 1-10 nF + 10 uF"
Changed lines of the file:
@@
 $EndComp
 $Comp
-L device:C_Small C10
+L Project:C C10
 U 1 1 58A85D67
 P 9800 5100
@@
 $EndComp
 $Comp
-L device:R_Small R3
+L Project:R R3
 U 1 1 58A9A2AE
 P 5700 2800
@@
 $EndComp
 $Comp
-L device:R_Small R1
+L Project:R R1
 U 1 1 58A9AA64
 P 5800 2100
@@
 $EndComp
 $Comp
-L device:R_Small R10
+L Project:R R10
 U 1 1 58A9B6EE
 P 9500 4900
@@
 $EndComp
 $Comp
-L device:R_Small R9
+L Project:R R9
 U 1 1 58A9DC80
 P 2700 4900
@@
 $EndComp
 $Comp
-L device:R_Small R12
+L Project:R R12
 U 1 1 58A9E677
 P 3350 5100
@@
 $EndComp
 $Comp
-L device:R_Small R13
+L Project:R R13
 U 1 1 58A9EAD2
 P 2200 5400
@@
 $EndComp
 $Comp
-L device:R_Small R17
+L Project:R R17
 U 1 1 58AA028C
 P 1900 5900
@@
 $EndComp
 $Comp
-L device:R_Small R16
+L Project:R R16
 U 1 1 58AA0F0C
 P 2600 5600
@@
 $EndComp
 $Comp
-L device:R_Small R6
+L Project:R R6
 U 1 1 58AA6BF1
 P 8900 3200
@@
 $EndComp
 $Comp
-L device:C_Small C8
+L Project:C C8
 U 1 1 58AC52BA
 P 2600 2100
@@
 $EndComp
 $Comp
-L device:C_Small C4
+L Project:C C4
 U 1 1 58AC5948
 P 4700 2100
@@
 $EndComp
 $Comp
-L device:C_Small C6
+L Project:C C6
 U 1 1 58AC7446
 P 7100 2950
@@
 $EndComp
 $Comp
-L device:R_Small R4
+L Project:R R4
 U 1 1 58AC810E
 P 7100 2650
@@
 $EndComp
 $Comp
-L device:L_Core_Iron L1
+L Device:L_Core_Iron L1
 U 1 1 58ACD441
 P 7600 2400
@@
 $EndComp
 $Comp
-L Transistor:BC817 T1
+L Transistor_BJT:BC817 T1
 U 1 1 58ACF046
 P 2900 5400
@@
 $EndComp
 $Comp
-L device:C_Small C12
+L Project:C C12
 U 1 1 58AD9379
 P 7900 5200
@@
 $EndComp
 $Comp
-L LibreSolar:Screw_Terminal_1x02 J3
+L Project:Screw_Terminal_1x02 J3
 U 1 1 58A7CE11
 P 10000 2800
@@
 $EndComp
 $Comp
-L LibreSolar:Screw_Terminal_1x02 J1
+L Project:Screw_Terminal_1x02 J1
 U 1 1 58A7E35A
 P 1650 2100
@@
 $EndComp
 $Comp
-L LibreSolar:Screw_Terminal_1x02 J2
+L Project:Screw_Terminal_1x02 J2
 U 1 1 58A7FE07
 P 6300 5800
@@
 $EndComp
 $Comp
-L device:CP_Small C2
+L Device:CP_Small C2
 U 1 1 58A857B0
 P 4000 2100
 F 0 "C2" H 4025 2175 50  0000 L CNN
 F 1 "1000u" H 4025 2025 50  0000 L CNN
-F 2 "Capacitors_THT:CP_Radial_D16.0mm_P7.50mm" H 4025 1875 50  0001 L CNN
+F 2 "Capacitor_THT:CP_Radial_D16.0mm_P7.50mm" H 4025 1875 50  0001 L CNN
 F 3 "" H 4025 2175 50  0000 C CNN
 F 4 "United Chemi-Con" H 600 300 50  0001 C CNN "Manufacturer"
@@
 $EndComp
 $Comp
-L device:CP_Small C5
+L Device:CP_Small C5
 U 1 1 58A85EB1
 P 8000 2800
 F 0 "C5" H 8020 2870 50  0000 L CNN
 F 1 "820u" H 8020 2720 50  0000 L CNN
-F 2 "Capacitors_THT:CP_Radial_D10.0mm_P5.00mm" H 8000 2800 50  0001 C CNN
+F 2 "Capacitor_THT:CP_Radial_D10.0mm_P5.00mm" H 8000 2800 50  0001 C CNN
 F 3 "" H 8000 2800 50  0000 C CNN
 F 4 "Panasonic" H 4200 1000 50  0001 C CNN "Manufacturer"
@@
 $EndComp
 $Comp
-L device:C_Small C3
+L Project:C C3
 U 1 1 58A8683F
 P 4400 2100
@@
 $EndComp
 $Comp
-L device:D_Small D1
+L Project:D D1
 U 1 1 58A87233
 P 4200 3000
@@
 $EndComp
 $Comp
-L device:Fuse_Small F1
+L Device:Fuse_Small F1
 U 1 1 58AA3600
 P 8900 2400
@@
 $EndComp
 $Comp
-L LibreSolar:+10V #PWR05
+L Project:+10V #PWR05
 U 1 1 58BE9B73
 P 2500 4800
@@
 $EndComp
 $Comp
-L LibreSolar:+10V #PWR06
+L Project:+10V #PWR06
 U 1 1 58BEA73B
 P 7900 4900
@@
 $EndComp
 $Comp
-L device:R_Small R2
+L Project:R R2
 U 1 1 58BEC59A
 P 3400 2800
@@
 $EndComp
 $Comp
-L LibreSolar:LM5107 U1
+L Project:LM5107 U1
 U 1 1 58C054FE
 P 8900 5200
@@
 $EndComp
 $Comp
-L LibreSolar:Q_NMOS Q1
+L Project:Q_NMOS Q1
 U 1 1 58C3E2A8
 P 6200 2100
@@
 $EndComp
 $Comp
-L LibreSolar:Q_NMOS Q4
+L Project:Q_NMOS Q4
 U 1 1 58C40039
 P 6200 2800
@@
 $EndComp
 $Comp
-L LibreSolar:Q_NMOS Q2
+L Project:Q_NMOS Q2
 U 1 1 58C41D81
 P 3000 2700
@@
 $EndComp
 $Comp
-L LibreSolar:Q_NMOS Q3
+L Project:Q_NMOS Q3
 U 1 1 58C43871
 P 3700 5800
@@
 BAT+
 $Comp
-L device:CP_Small C1
+L Device:CP_Small C1
 U 1 1 59108F15
 P 3600 2100
 F 0 "C1" H 3625 2175 50  0000 L CNN
 F 1 "1000u" H 3625 2025 50  0000 L CNN
-F 2 "Capacitors_THT:CP_Radial_D16.0mm_P7.50mm" H 3625 1875 50  0001 L CNN
+F 2 "Capacitor_THT:CP_Radial_D16.0mm_P7.50mm" H 3625 1875 50  0001 L CNN
 F 3 "" H 3625 2175 50  0000 C CNN
 F 4 "United Chemi-Con" H 200 300 50  0001 C CNN "Manufacturer"
@@
 $EndComp
 Wire Wire Line
-	7900 4900 7900 5100
+	7900 4900 7900 5000
 Wire Wire Line
 	8600 5000 7900 5000
@@
 	2500 4900 2600 4900
 Wire Wire Line
-	9000 2400 9700 2400
-Wire Wire Line
-	9000 3200 9700 3200
+	9000 2400 9400 2400
+Wire Wire Line
+	9000 3200 9100 3200
 Wire Wire Line
 	1700 5900 1800 5900
@@
 	2600 2000 2600 1700
 Wire Wire Line
-	7750 2400 8800 2400
+	7750 2400 8000 2400
 Wire Wire Line
 	8600 2400 8600 2300
@@
 	8600 5400 7900 5400
 Wire Wire Line
-	7900 5300 7900 5500
+	7900 5300 7900 5400
 Wire Wire Line
 	6700 3300 6700 3200
@@
 	9800 4900 9800 5000
 Wire Wire Line
-	3000 4900 3000 5200
+	3000 4900 3000 5100
 Wire Wire Line
 	3000 5100 3250 5100
@@
 	2800 4900 3000 4900
 Wire Wire Line
-	2300 5400 2700 5400
+	2300 5400 2600 5400
 Wire Wire Line
 	2600 5400 2600 5500
@@
 	2500 4800 2500 4900
 Wire Wire Line
-	2300 1700 6300 1700
+	2300 1700 2600 1700
 Wire Wire Line
 	5900 2100 6000 2100
@@
 	3400 2900 3400 3000
 Wire Wire Line
-	6300 2400 7450 2400
+	6300 2400 7100 2400
 Wire Wire Line
 	6100 5700 6000 5700
@@
 	6300 1700 6300 1900
 Wire Wire Line
-	5800 2800 6000 2800
+	5800 2800 5900 2800
 Wire Wire Line
 	5900 3000 5900 2800
@@
 	4300 3000 5900 3000
 Wire Wire Line
-	6300 2300 6300 2600
+	6300 2300 6300 2400
 Wire Wire Line
 	6300 3200 6300 3000
 Wire Wire Line
-	2300 2600 2800 2600
-Wire Wire Line
-	3200 2600 4800 2600
+	2300 2600 2600 2600
+Wire Wire Line
+	3200 2600 3400 2600
 Wire Wire Line
 	3000 2900 3000 3000
 Wire Wire Line
-	3000 3000 4100 3000
-Wire Wire Line
-	3900 5900 6100 5900
-Wire Wire Line
-	2000 5900 3500 5900
-Wire Wire Line
-	3700 5100 3700 5600
+	3000 3000 3400 3000
+Wire Wire Line
+	3900 5900 4100 5900
+Wire Wire Line
+	2000 5900 2100 5900
+Wire Wire Line
+	3700 5100 3700 5300
 Wire Wire Line
 	5400 1700 5400 1600
@@
 Connection ~ 8000 3200
 Wire Wire Line
-	6300 3200 8800 3200
+	6300 3200 6700 3200
 Wire Wire Line
 	7100 2400 7100 2550
@@
 	7100 2750 7100 2850
 $Comp
-L device:D_Zener_Small D5
+L Device:D_Zener_Small D5
 U 1 1 5A2D4B0C
 P 5200 5700
@@
 	6000 5700 6000 5500
 Wire Wire Line
-	5100 5500 6000 5500
+	5100 5500 5200 5500
 Wire Wire Line
 	5200 5600 5200 5500
@@
 Connection ~ 5200 5900
 $Comp
-L device:C_Small C7
+L Project:C C7
 U 1 1 5A2E653B
 P 9400 2800
@@
 Connection ~ 9400 3200
 $Comp
-L device:C_Small C27
+L Project:C C27
 U 1 1 5A314523
 P 5700 5700
@@
 Connection ~ 5700 5900
 $Comp
-L device:C_Small C28
+L Project:C C28
 U 1 1 5A336B6E
 P 4100 5600
@@
 	4100 5700 4100 5900
 Connection ~ 4100 5900
+Wire Wire Line
+	7900 5000 7900 5100
+Wire Wire Line
+	3000 5900 3500 5900
+Wire Wire Line
+	2600 5900 3000 5900
+Wire Wire Line
+	2600 1700 3600 1700
+Wire Wire Line
+	8600 2400 8800 2400
+Wire Wire Line
+	7900 5400 7900 5500
+Wire Wire Line
+	6700 3200 7100 3200
+Wire Wire Line
+	4000 2600 4400 2600
+Wire Wire Line
+	4700 2600 4800 2600
+Wire Wire Line
+	4400 2600 4700 2600
+Wire Wire Line
+	3400 2600 3600 2600
+Wire Wire Line
+	3400 3000 4100 3000
+Wire Wire Line
+	3000 5100 3000 5200
+Wire Wire Line
+	2600 5400 2700 5400
+Wire Wire Line
+	2600 2600 2800 2600
+Wire Wire Line
+	4700 1700 5400 1700
+Wire Wire Line
+	4400 1700 4700 1700
+Wire Wire Line
+	4000 1700 4400 1700
+Wire Wire Line
+	5900 2800 6000 2800
+Wire Wire Line
+	6300 2400 6300 2600
+Wire Wire Line
+	5400 1700 6300 1700
+Wire Wire Line
+	2100 5900 2600 5900
+Wire Wire Line
+	8700 3200 8800 3200
+Wire Wire Line
+	9100 3200 9400 3200
+Wire Wire Line
+	3600 1700 4000 1700
+Wire Wire Line
+	3600 2600 4000 2600
+Wire Wire Line
+	8000 2400 8600 2400
+Wire Wire Line
+	8000 3200 8700 3200
+Wire Wire Line
+	7100 2400 7450 2400
+Wire Wire Line
+	7100 3200 8000 3200
+Wire Wire Line
+	5200 5500 5700 5500
+Wire Wire Line
+	5200 5900 5700 5900
+Wire Wire Line
+	9400 2400 9700 2400
+Wire Wire Line
+	9400 3200 9700 3200
+Wire Wire Line
+	5700 5500 6000 5500
+Wire Wire Line
+	5700 5900 6100 5900
+Wire Wire Line
+	3700 5300 3700 5600
+Wire Wire Line
+	4100 5900 5200 5900
+Text Notes 2250 1200 0    50   ~ 0
+typisch: 1-10 nF + 10 uF
 $EndSCHEMATC
