File: interfaces.sch (KiCad schematic (older format))
At the start: 32 parts, among them J4 UEXT, P3 USB Micro B, Q5 BSS84, Q6 BSS84, Q7 BSS84, T3 MMBT3904, T4 MMBT3904, U8 TJA1042T/3

Commit message: Final version for Jan/2018 production
Parts:
- D3: value USBLC6-2SC6 -> USBLC6-2SC6Y; PartNumber USBLC6-2SC6 -> USBLC6-2SC6Y
- D4: Alternative (none) -> SZNUP2105L
- F2, F3: Manufacturer Bel Fuse -> Bel
Changed lines of the file:
@@
 Sheet 5 6
 Title "MPPT Charger 20A"
-Date "2017-12-11"
-Rev "0.9"
+Date "2018-01-18"
+Rev "0.10"
 Comp ""
 Comment1 "Author: Martin Jäger"
@@
 F 4 "ON Semiconductor" H -250 500 50  0001 C CNN "Manufacturer"
 F 5 "NUP2105LT1G" H -250 500 50  0001 C CNN "PartNumber"
+F 6 "SZNUP2105L" H 9900 2200 60  0001 C CNN "Alternative"
 	1    9900 2200
 	1    0    0    -1
@@
 P 3600 2400
 F 0 "D3" H 3350 2750 50  0000 C CNN
-F 1 "USBLC6-2SC6" H 3600 2050 50  0000 C CNN
+F 1 "USBLC6-2SC6Y" H 3600 2050 50  0000 C CNN
 F 2 "LibreSolar:SOT-23-6" H 4250 2750 50  0001 C CNN
 F 3 "" H 3350 2750 50  0001 C CNN
 F 4 "STMicroelectronics" H 450 350 50  0001 C CNN "Manufacturer"
-F 5 "USBLC6-2SC6" H 450 350 50  0001 C CNN "PartNumber"
+F 5 "USBLC6-2SC6Y" H 450 350 50  0001 C CNN "PartNumber"
 	1    3600 2400
 	-1   0    0    -1
@@
 F 2 "LibreSolar:R_1206_3216" H 2800 1600 50  0001 L CNN
 F 3 "" H 2750 1800 50  0001 C CNN
-F 4 "Bel Fuse" H 150 -100 60  0001 C CNN "Manufacturer"
+F 4 "Bel" H 150 -100 60  0001 C CNN "Manufacturer"
 F 5 "0ZCJ0020FF2E" H 150 -100 60  0001 C CNN "PartNumber"
 	1    2750 1800
@@
 F 2 "LibreSolar:R_1206_3216" H 9000 4800 50  0001 L CNN
 F 3 "" H 8950 5000 50  0001 C CNN
-F 4 "Bel Fuse" H 1250 0   60  0001 C CNN "Manufacturer"
+F 4 "Bel" H 1250 0   60  0001 C CNN "Manufacturer"
 F 5 "0ZCJ0020FF2E" H 1250 0   60  0001 C CNN "PartNumber"
 	1    8950 5000

Commit message: Update to KiCad 5 schematic library
Parts:
- C25, C26, C39: symbol device:C_Small -> Project:C
- D10, D9: symbol device:D_Small -> Project:D
- D3: symbol LibreSolar:USBLC6-2SC6 -> Project:USBLC6-2SC6
- D4: symbol LibreSolar:NUP2105L -> Project:NUP2105L
- D8: symbol device:D_Zener_Small -> Device:D_Zener_Small
- F2, F3: symbol device:Polyfuse -> Device:Polyfuse
- J4: symbol LibreSolar:UEXT -> Project:UEXT
- JP1, JP2: symbol LibreSolar:RJ45_NS -> Project:RJ45_NS
- JP3: footprint Pin_Headers:Pin_Header_Angled_1x02_Pitch2.54mm -> Connector_PinHeader_2.54mm:PinHeader_1x02_P2.54mm_Horizontal; symbol device:Jumper_NC_Small -> Device:Jumper_NC_Small
- Q5, Q6, Q7: symbol device:Q_PMOS_GSD -> Device:Q_PMOS_GSD
- R30, R33, R34, R35, R36, R38, R46, R47, R48, R49, R5: symbol device:R_Small -> Project:R
- T3, T4: symbol Transistor:BC817 -> Transistor_BJT:BC817
- U8: symbol LibreSolar:TJA1042T-3 -> Project:TJA1042T-3
Other:
- note added: "ToDo: check R47 \n--> should be smaller?"
- note removed: "ToDo: check R47 --> should be smaller?"
Changed lines of the file:
@@
 $EndComp
 $Comp
-L device:C_Small C39
+L Project:C C39
 U 1 1 58BE3440
 P 6300 2100
@@
 $EndComp
 $Comp
-L device:C_Small C26
+L Project:C C26
 U 1 1 58BE3447
 P 6000 2100
@@
 $EndComp
 $Comp
-L device:R_Small R36
+L Project:R R36
 U 1 1 58BE344E
 P 8900 2300
@@
 $EndComp
 $Comp
-L LibreSolar:RJ45_NS JP1
+L Project:RJ45_NS JP1
 U 1 1 58BE345B
 P 7050 3650
@@
 $EndComp
 $Comp
-L LibreSolar:TJA1042T-3 U8
+L Project:TJA1042T-3 U8
 U 1 1 58BE3467
 P 7700 2200
@@
 $EndComp
 $Comp
-L device:Jumper_NC_Small JP3
+L Device:Jumper_NC_Small JP3
 U 1 1 58BE3476
 P 8900 2000
 F 0 "JP3" H 8900 2080 50  0000 C CNN
 F 1 "Jumper_NC_Small" H 8910 1940 50  0001 C CNN
-F 2 "Pin_Headers:Pin_Header_Angled_1x02_Pitch2.54mm" H 8900 2000 50  0001 C CNN
+F 2 "Connector_PinHeader_2.54mm:PinHeader_1x02_P2.54mm_Horizontal" H 8900 2000 50  0001 C CNN
 F 3 "" H 8900 2000 50  0001 C CNN
 	1    8900 2000
@@
 $EndComp
 $Comp
-L LibreSolar:RJ45_NS JP2
+L Project:RJ45_NS JP2
 U 1 1 58BE348A
 P 8850 3650
@@
 $EndComp
 $Comp
-L device:R_Small R35
+L Project:R R35
 U 1 1 58BE3F9C
 P 5150 4700
@@
 $EndComp
 $Comp
-L device:R_Small R34
+L Project:R R34
 U 1 1 58BE3FA3
 P 4800 4700
@@
 $EndComp
 $Comp
-L LibreSolar:UEXT J4
+L Project:UEXT J4
 U 1 1 58BDEEA0
 P 2600 4900
@@
 $EndComp
 $Comp
-L LibreSolar:NUP2105L D4
+L Project:NUP2105L D4
 U 1 1 58BE0956
 P 9900 2200
@@
 $EndComp
 $Comp
-L LibreSolar:USBLC6-2SC6 D3
+L Project:USBLC6-2SC6 D3
 U 1 1 58BE3F7F
 P 3600 2400
@@
 $EndComp
 $Comp
-L device:C_Small C25
+L Project:C C25
 U 1 1 58CC2EC7
 P 1900 2850
@@
 $EndComp
 $Comp
-L device:R_Small R46
+L Project:R R46
 U 1 1 58CC345E
 P 2700 2600
@@
 $EndComp
 $Comp
-L device:Polyfuse F2
+L Device:Polyfuse F2
 U 1 1 592A398B
 P 2750 1800
@@
 RJ45_5
 $Comp
-L device:Polyfuse F3
+L Device:Polyfuse F3
 U 1 1 5954FB5B
 P 8950 5000
@@
 $EndComp
 $Comp
-L device:D_Small D9
+L Project:D D9
 U 1 1 595501B6
 P 9400 5000
@@
 $EndComp
 $Comp
-L device:D_Small D10
+L Project:D D10
 U 1 1 595502E8
 P 9400 5400
@@
 5V signal output
 $Comp
-L device:Q_PMOS_GSD Q5
+L Device:Q_PMOS_GSD Q5
 U 1 1 59558C66
 P 3600 6400
@@
 5V_OUT
 $Comp
-L device:R_Small R33
+L Project:R R33
 U 1 1 5955A770
 P 3200 6500
@@
 $EndComp
 $Comp
-L device:R_Small R38
+L Project:R R38
 U 1 1 5955A862
 P 3000 6700
@@
 $EndComp
 $Comp
-L device:R_Small R47
+L Project:R R47
 U 1 1 5955A8AC
 P 2300 7000
@@
 $EndComp
 $Comp
-L Transistor:BC817 T4
+L Transistor_BJT:BC817 T4
 U 1 1 5955C30A
 P 2700 7000
@@
 	3600 6700 3600 6600
 Wire Wire Line
-	3100 6700 3600 6700
+	3100 6700 3200 6700
 Wire Wire Line
 	3200 6400 3200 6300
 Wire Wire Line
-	3000 6300 3400 6300
+	3000 6300 3200 6300
 Wire Wire Line
 	3000 6300 3000 6200
@@
 	1900 2950 1900 3000
 Wire Wire Line
-	2300 2000 3000 2000
+	2300 2000 2500 2000
 Wire Wire Line
 	2500 1800 2500 2000
@@
 DCDC_OUT
 $Comp
-L device:Q_PMOS_GSD Q6
+L Device:Q_PMOS_GSD Q6
 U 1 1 5A2F2F44
 P 1900 4400
@@
 UEXT_EN
 Wire Wire Line
-	1500 4400 1700 4400
-Wire Wire Line
-	2000 4000 2000 4200
+	1500 4400 1600 4400
+Wire Wire Line
+	2000 4000 2000 4100
 Wire Wire Line
 	2000 4600 2000 4700
@@
 	2000 4700 2200 4700
 $Comp
-L device:R_Small R5
+L Project:R R5
 U 1 1 5A30156C
 P 1800 4100
@@
 	1600 4100 1600 4400
 Connection ~ 1600 4400
-Text Notes 3500 8700 0    100  ~ 0
-ToDo: check R47 --> should be smaller?
-$Comp
-L device:Q_PMOS_GSD Q7
+Text Notes 1200 7450 0    50   ~ 0
+ToDo: check R47 \n--> should be smaller?
+$Comp
+L Device:Q_PMOS_GSD Q7
 U 1 1 5A44CCDC
 P 8200 5100
@@
 $EndComp
 $Comp
-L device:R_Small R49
+L Project:R R49
 U 1 1 5A44CCF0
 P 7300 5200
@@
 $EndComp
 $Comp
-L device:R_Small R30
+L Project:R R30
 U 1 1 5A44CCF9
 P 7100 5400
@@
 $EndComp
 $Comp
-L device:R_Small R48
+L Project:R R48
 U 1 1 5A44CD05
 P 6400 5700
@@
 $EndComp
 $Comp
-L Transistor:BC817 T3
+L Transistor_BJT:BC817 T3
 U 1 1 5A44CD0E
 P 6800 5700
@@
 	8200 5400 8200 5300
 Wire Wire Line
-	7200 5400 8200 5400
+	7200 5400 7300 5400
 Wire Wire Line
 	7300 5100 7300 5000
 Wire Wire Line
-	6700 5000 8000 5000
+	6700 5000 7300 5000
 Connection ~ 7300 5000
 $Comp
@@
 V_BUS_EN
 $Comp
-L device:D_Zener_Small D8
+L Device:D_Zener_Small D8
 U 1 1 5A44E18E
 P 7600 5200
@@
 Text Notes 5100 7600 0    50   ~ 0
 If not stated otherwise, all MLCC 50V X7R
+Wire Wire Line
+	3200 6300 3400 6300
+Wire Wire Line
+	3200 6700 3600 6700
+Wire Wire Line
+	2500 2000 3000 2000
+Wire Wire Line
+	2000 4100 2000 4200
+Wire Wire Line
+	1600 4400 1700 4400
+Wire Wire Line
+	7300 5000 7600 5000
+Wire Wire Line
+	7300 5400 7600 5400
+Wire Wire Line
+	7600 5000 8000 5000
+Wire Wire Line
+	7600 5400 8200 5400
 $EndSCHEMATC
